File: MagicThings/Lume2/lume2_hw/lume2.sch (KiCad schematic (older format))
At the start: 41 parts, among them M1 MOTOR, Q1 NPN, Q2 NPN, SW1 BUTTON, SW2 BUTTON, SW3 BUTTON

Commit message: 
Parts:
- removed BZ1: BUZZER, symbol BUZZER
- removed C15, C16, C17, C26: 0.1u, symbol C
- removed C18: 4.7u, symbol C
- removed C19, C27, C28, C29: 1u, symbol C
- removed C20, C21: 6.8pF, symbol C
- removed C22, C23: 10u, symbol C
- removed C24: 10u, CAP_0805, symbol C
- removed C25: 0.1u, CAP_0603, symbol C
- removed D1: 1N4148, SOD323, symbol DIODE
- removed DA1: BQ24010, symbol BQ24010
- removed DD3: M24C02, TSSOP8, symbol EEPROM_I2C
- removed M1: MOTOR, symbol MOTOR
- removed Q1, Q2: NPN, symbol NPN
- added C1, C10, C6: 4.7u, CAP_0603, symbol C
- added C11, C2, C3, C4, C5: 0.1u, CAP_0603, symbol C
- added C12, C13, C7: 1u, CAP_0603, symbol C
- added C8, C9: 6.8pF, CAP_0603, symbol C
- added D1: SS14, SMA, symbol D_SHOTTKY
- added DD1, DD3: PCA9635, symbol PCA9635
- added FU1, FU2, FU3, FU4: SOLDERFUSE, symbol SOLDERFUSE
- added HOLE1, HOLE2, HOLE3, HOLE4: HOLE_METALLED, symbol HOLE_METALLED
- added R1, R11, R12, R13, R14, R15, R16, R17, R18, R19, R20, R21, R22, R23, R24, R25, R26, R27, R28, R29, R30, R31, R33: 100R, RES_0603, symbol R
- added R32, R34: 4k7, RES_0603, symbol R
- added XL1: CONN_3, symbol CONN_3
- added XL10: CONN_1, symbol CONN_1
- added XL2, XL4, XL5, XL6: CONN_10, symbol CONN_10
- added XL3: CONN_NOKIA_LCD, symbol CONN_NOKIA_LCD
- added XL8: CONN_2, symbol CONN_2
- B1: footprint BAT_LP383450 -> CR2032
- R10: value 1.5k -> 100R; footprint (none) -> RES_0603
- R2, R3: value 4k7 -> 100R; footprint (none) -> RES_0603
- R4, R5: value 1k -> 100R; footprint (none) -> RES_0603
- R6: value 1.8k* -> 100R; footprint (none) -> RES_0603
- R7, R9: value 100k -> 100R; footprint (none) -> RES_0603
- R8: value 3.9k* -> 100R; footprint (none) -> RES_0603
- renumbered DA2 to DA1, DA3 to DA2, XL2 to XL7, XL4 to XL9, XTAL2 to XTAL1
Connections:
- net labels added: FU0, FU1, FU2, FU3, LED_OE
- net labels removed: +BATT, BuzzerIn, BuzzerOut, CC_CS, CC_GDO0, CC_GDO2, CC_MISO, CC_MOSI, CC_SCK, CHRG, CHRG_DONE, I2C_PullUp, MotorIn, MotorOut, PWR_GOOD, UBat/2
- wire segments 157 -> 288
- no-connect marks 9 -> 16
Other:
- note added: "Address\nsetting"
- note added: "Battery 4.5V\n(3xAA)"
- note added: "LCD"
- note added: "LEDs controller\nI2C addr = 0x1A"
- note added: "LEDs controller\nI2C addr = 0x2B"
- note added: "Luminocity\nsensor"
- note removed: "Battery\nmeter"
- note removed: "I2C Addr = 1010 (A2)(A1)(A0) = 1010 111"
- note removed: "Li-Ion charger\n1.5k => 0.56 A"
- moved on the sheet: B1, DA1, DA2, DD2, SW1, SW2, SW3, XL7, XL9, XTAL1
