File: Armlet/Armlet3/Armlet3_hw/Armlet3.kicad_pcb (KiCad board)
At the start: 2 copper layers, 74 x 40.5 mm, 155 parts, among them M1 MOTOR, Q1 MMBT2222, Q2 MMBT2222, Q3 TSOP75256, Q4 IRLML9303, Q6 MMBT2222, Q7 BC848CL, SW1 BUTTON, SW2 BUTTON, SW3 BUTTON, SW4 BUTTON, SW5 BUTTON, SW6 BUTTON, SW7 BUTTON, SW8 BUTTON, SW9 BUTTON

Commit message: Pcb repaired. BOM modified. Radio works.
Parts:
- C18: renamed from ?; value 1u -> 0.1u
- C19: renamed from ?; value 0.1u -> 1u
- C26, C27: value 4.7u -> 10u
- C29: value 1u -> DNM
- C62: renamed from ?; value * -> 3.3pF
- C63: renamed from ?; value * -> 6.8pF
- C7, C9: value 0.01u -> 10n
- DA1: value NCP583SQ -> DNM
- L8: renamed from ?; value * -> 15nH
- Q7: value BC848CL -> DNM
- R15: value 1k -> DNM
- R16: value 10k -> DNM
- R7, R9: value 390k -> 330k
- TP2, TP3: renamed from ?; value (none) -> TESTPOINT
- gave numbers to parts that had none: 47
