File: Lockets/Tirusse2/Tirusse2_hw/Tirusse2.sch (KiCad schematic (older format))
At the start: 142 parts, among them M1 MOTOR, Q1 MMBT2222, Q2 MMBT2222, Q3 TSOP75256, Q5 BC848CL, Q6 MMBT2222, Q7 DNM, SW1 BUTTON, SW2 BUTTON, SW3 BUTTON, SW4 BUTTON, SW5 BUTTON, SW6 BUTTON, SW7 BUTTON, SW8 BUTTON, SW9 BUTTON

Commit message: 
Parts:
- removed ANT1: ANT_PCB_MONO, symbol ANT_PCB_MONO
- removed BZ1: BUZZER, symbol BUZZER
- removed C13: 47n, symbol C
- removed C20, C21, C42, C47, C52: 0.1u, CAP_0402, symbol C
- removed C22, C23, C25, C30, C32, C33, C34, C51, C56, C57: 0.1u, CAP_0603, symbol C
- removed C24, C31, C35: 10u, CAP_0805, symbol C
- removed C36, C37, C55: 20pF, CAP_0402, symbol C
- removed C45, C60, C61: 0.1u, symbol C
- removed C48, C64: 1u, symbol C
- removed C49, C54: 1u, CAP_0402, symbol C
- removed C50: 10u, symbol C
- removed C53: 100pF, CAP_0402, symbol C
- removed C58: 150pF, CAP_0402, symbol C
- removed C59: 1n, CAP_0402, symbol C
- removed C62: 3.3pF, symbol C
- removed C63: 6.8pF, symbol C
- removed D3: PMLL4148, symbol DIODE
- removed DA2: VS1011, symbol VS1011
- removed DA3: MAX4453, symbol GENERIC_8PIN
- removed DA5: NCP583SQ, symbol NCP583SQ
- removed DD3: MMA8452Q, symbol MMA8452Q
- removed HOLE1, HOLE2: HOLE_METALLED, symbol HOLE_METALLED
- removed M1: MOTOR, symbol MOTOR
- removed Q1, Q2, Q6: MMBT2222, symbol NPN
- removed Q3: TSOP75256, symbol TSOP752XX
- removed Q5: BC848CL, symbol NPN
- removed Q7: DNM, symbol NPN
- removed R11, R6: 20, symbol R
- removed R14: 220R, RES_0402, symbol R
- removed R15, R16: DNM, RES_0402, symbol R
- removed R17, R26, R27, R30, R32, R34: 10k, RES_0402, symbol R
- removed R18: 51R, RES_0402, symbol R
- removed R20: 100, symbol R
- removed R21: 150, RES_0402, symbol R
- removed R25: 100, RES_0402, symbol R
- removed R28, R33: 1k, RES_0603, symbol R
- removed R29, R35: 1k, RES_0402, symbol R
- removed R36: 20k, RES_0402, symbol R
- removed R37: 330k, RES_0402, symbol R
- removed R39, R4, R5: 1k, symbol R
- removed R8: 10, symbol R
- removed SW1, SW2, SW3, SW4, SW5, SW6, SW7, SW8, SW9: BUTTON, symbol BUTTON
- removed VCap1, VCap2: 2.2u, CAP_0402, symbol C
- removed XL11: CONN_NOKIA_BAT, symbol CONN_NOKIA_BAT
- removed XL2: CONN_AUDIO_SIMPLE, symbol CONN_AUDIO_SIMPLE
- added C13: 100u, symbol CP
- added C18: 20pF, CAP_0402, symbol C
- added D1: BAT54WS, symbol D_SHOTTKY
- added D3: BAXXXC, symbol BAXXXC
- added DD2: STM32F10X-48, ~, symbol STM32F10X-48
- added F1, F2, F3, F4, F5, F6, F7: FUSE0R, symbol FUSE0R
- added Q1: IRLML6302, symbol IRLML6302
- added SW1: SWITCH, symbol SWITCH
- added XL1, XL4, XL8: CONN_1, ~, symbol CONN_1
- added XL2, XL3: CONN_1, symbol CONN_1
- C12: value 10n -> 1u; footprint (none) -> CAP_0603
- C15: value 10n -> 20pF; footprint (none) -> CAP_0402
- C29: value DNM -> 1u
- DA1: value DNM -> NCP583SQ
- L7: value 100uH -> 22uH
- L8: value 15nH -> 22uH; footprint IND_0402 -> IND_1812
- R2: value 4k7 -> *; footprint (none) -> RES_0603
- R3: value 4k7 -> 220R; footprint (none) -> RES_0402
Connections:
- net labels added: BAT, Debug, PWR_IN, RX1, TX1
- net labels removed: 12MHz_Clk, ACC_IRQ, AGND, Btn1, Btn2, Btn3, Btn4, Btn5, Btn6, Btn7, Btn8, Btn9, Buzzer, BuzzerOut, I2C_SCL, I2C_SDA, LCD_BCKLT, LCD_DA0, LCD_DA1, LCD_DA2, LCD_DA3, LCD_DA4, LCD_DA5, LCD_DA6, LCD_DA7, LCD_DC, LCD_RD, LCD_WR, LCD_XCS, LCD_XRES, P_SCL, P_SDA, PeriphPwr, RX2, SD_CLK, SD_CMD, SD_DAT0, SD_DAT1, SD_DAT2, SD_DAT3, SD_POWER, SND_C, SND_L, SND_R, TX2, USB_DM, USB_DP, VS_DREQ, VS_RST, VS_SCLK, VS_SI, VS_SO, VS_XCS, VS_XDCS, Vibro, VibroOut, XLed1, XLed2, XotarIn, XotarLED, XotarPower, klNFC_Rx, klNFC_Tx, klNFC_Vcc
- wire segments 432 -> 191
- no-connect marks 18 -> 19
Other:
- note added: "3.0V 150mA power regulator"
- note added: "Address\nsettings"
- note added: "Battery"
- note removed: "100pF & 10k => \nf0=160 kHz \n"
- note removed: "20pF cap removes\nremains of carrier"
- note removed: "3.3V 150mA power regulator"
- note removed: "Accelerometer\nI2C addr = 0x1C"
- note removed: "Audio"
- note removed: "Buttons"
- note removed: "Half-Vcc divider"
- note removed: "I2C and Accelerometer"
- note removed: "I2C pull-ups"
- note removed: "Matching circuit"
- note removed: "Nokia battery \nconnector"
- note removed: "Note AGND here ^^^"
- note removed: "Vibro & buzzer"
- note removed: "Xotar in & out"
- note removed: "klNFC"
- moved on the sheet: C26, C27, C28, C29, C38, C39, C40, C41, C43, C44, DA1, DA4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
