File: SciFi/IrGirandole/Girandole_hw/girandole.kicad_pcb (KiCad board)
At the start: 2 copper layers, 110 x 23 mm, 72 parts, among them Q1 IRLML6302, SW1 SWITCH

Commit message: 
Parts:
- removed C1: 100pF, CAP_0402
- removed C10, C14, C38, C39, C40, C43, C44: 0.1u, CAP_0402
- removed C11, C6: 220pF, CAP_0402
- removed C12, C28, C29: 1u, CAP_0402
- removed C13: 100u, CAP_06xxR
- removed C15, C18: 20pF, CAP_0402
- removed C16, C17: 10pF, CAP_0402
- removed C2, C4: 1.5pF, CAP_0402
- removed C26, C27, C41: 10u, CAP_0805
- removed C3: 1pF, CAP_0402
- removed C5, C8: 3.3pF, CAP_0402
- removed C7, C9: 10n, CAP_0402
- removed D1: BAT54WS, DIODE_SOD323
- removed D2: LED, LED-3MM
- removed D3: BAXXXC, SOT23
- removed DA1: NCP583SQ, SC82AB
- removed DA4: MCP73832, SOT23-5
- removed DD1: CC1101, QFN20
- removed DD2: STM32F10X-48, LQFP48
- removed F1, F2, F3, F4, F5, F6, F7: FUSE0R, SMD0603_FUSE
- removed L1, L6: 18nH, IND_0402
- removed L2, L3, L4, L5: 12nH, IND_0402
- removed L7: 22uH, IND_1210
- removed L8: 22uH, IND_HOLE_M
- removed Q1: IRLML6302, SOT23
- removed R1: 56k, RES_0402
- removed R10: 2k, RES_0402
- removed R19: 1k, RES_0402
- removed R2: *, RES_0603
- removed R3: 220R, RES_0402
- removed R7, R9: 330k, RES_0402
- removed SW1: SWITCH, SIL-3
- removed TP2, TP3: TESTPOINT, TESTPOINT_1MM
- removed XL1, XL4, XL7, XL8: CONN_1, SIL-1
- removed XL10: USB_MICRO_B, USB_KMMX_ABSMT5SG_30TR
- removed XL2, XL3: CONN_1, SIL1_SQUARE_4MM
- removed XL5: CONN_3, SIL-3
- removed XL6: ST_SWD, SIL-4
- removed XTAL1: 27MHz, CRYSTAL_03225C4
- removed XTAL2: 12.0MHz, CRYSTAL_0503x4-4
Routing:
- net GND: track 449.7 -> 0.00 mm, vias 63 -> 0
- net +3.3V: track 180.8 -> 0.00 mm, vias 11 -> 0
- net +BATT: track 107.1 -> 0.00 mm
- net /Charge: track 96.2 -> 0.00 mm, vias 2 -> 0
- net N-000007: track 91.6 -> 0.00 mm, vias 2 -> 0
- net /UBat_2: track 83.4 -> 0.00 mm, vias 2 -> 0
- net N-0000049: track 30.0 -> 0.00 mm, vias 1 -> 0
- net N-0000048: track 29.3 -> 0.00 mm
- net +5V: track 21.6 -> 0.00 mm, vias 2 -> 0
- net N-0000038: track 15.5 -> 0.00 mm, vias 2 -> 0
- net /CC_CS: track 14.8 -> 0.00 mm
- net /SWCLK: track 11.0 -> 0.00 mm
- net /CC_GDO0: track 11.0 -> 0.00 mm, vias 2 -> 0
- net /CC_GDO2: track 8.34 -> 0.00 mm
- net /PWR_IN: track 8.06 -> 0.00 mm
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- removed copper zone on B.Cu, net GND
- removed copper zone on F.Cu, net GND
Other:
- board outline removed

Commit message: Girandole hw completed
Parts:
- added BZ1: BUZZER, BUZZER_HC0903, F.Cu at (267.8, 169.0)
- added C1: 3.3pF, CAP_0603, F.Cu at (268.0, 179.2)
- added C10: 1n, CAP_0603, F.Cu at (263.8, 199.4)
- added C11: 0.1u, CAP_0603, F.Cu at (268.0, 185.0)
- added C15: 20pF, CAP_0603, F.Cu at (259.0, 194.3)
- added C18: 20pF, CAP_0603, F.Cu at (259.0, 202.3)
- added C2: 0.1u, CAP_0603, F.Cu at (259.1, 165.2)
- added C3: 1000u, CAP_10xxR, F.Cu at (246.8, 169.4)
- added C38: 0.1u, CAP_0603, F.Cu at (244.8, 190.4)
- added C39: 0.1u, CAP_0603, F.Cu at (241.2, 200.1)
- added C40: 0.1u, CAP_0603, F.Cu at (252.8, 204.4)
- added C41: 10u, CAP_0805, F.Cu at (242.8, 190.0)
- added C43: 0.1u, CAP_0603, F.Cu at (254.2, 201.8)
- added C44: 0.1u, CAP_0603, F.Cu at (254.4, 195.4)
- added C5: 0.1u, CAP_0603, F.Cu at (246.8, 171.4)
- added C6: 1n, CAP_0603, F.Cu at (265.6, 205.2)
- added C7: 1u, CAP_0603, F.Cu at (262.0, 205.2)
- added C8: 10u, CAP_0805, F.Cu at (260.0, 205.6)
- added C9: 1u, CAP_0603, F.Cu at (265.6, 199.4)
- added D1: LED, LED0603, F.Cu at (257.0, 188.4)
- added D2: LED, LED-5MM, F.Cu at (253.4, 175.0)
- added D3: LED, LED-5MM, F.Cu at (260.4, 175.0)
- added D4: LED, LED-5MM, F.Cu at (253.4, 181.8)
- added D5: LED, LED-5MM, F.Cu at (260.4, 181.8)
- added DA1: MAX4453, SOT23-8, F.Cu at (268.0, 182.2)
- added DA2: LP2951, SO8E, F.Cu at (269.4, 203.0)
- added DD2: STM32F10X-48, LQFP48, F.Cu at (247.8, 197.8)
- added F1: FUSE0R, SMD0603_FUSE, F.Cu at (242.4, 207.4)
- added F2: FUSE0R, SMD0603_FUSE, F.Cu at (244.0, 207.4)
- added F3: FUSE0R, SMD0603_FUSE, F.Cu at (245.6, 207.4)
- added F4: FUSE0R, SMD0603_FUSE, F.Cu at (247.2, 207.4)
- added F5: FUSE0R, SMD0603_FUSE, F.Cu at (248.8, 207.4)
- added F6: FUSE0R, SMD0603_FUSE, F.Cu at (250.4, 207.4)
- added F7: FUSE0R, SMD0603_FUSE, F.Cu at (252.0, 207.4)
- added F8: FUSE0R, SMD0603_FUSE, F.Cu at (257.0, 172.6)
- added HOLE1: HOLE_METALLED, Hole3_5_out6mm, F.Cu at (276.0, 167.5)
- added HOLE2: HOLE_METALLED, Hole3_5_out6mm, F.Cu at (238.0, 167.5)
- added HOLE3: HOLE_METALLED, Hole3_5_out6mm, F.Cu at (276.0, 205.5)
- added HOLE4: HOLE_METALLED, Hole3_5_out6mm, F.Cu at (238.0, 205.5)
- added Q1: TSOP752XX, TSOP752, F.Cu at (257.4, 167.8)
- added Q2: LED_RGB 5050, LED_HH5050_RGB, F.Cu at (257.0, 188.4)
- added Q3: TSOP48XX, SIL-3, F.Cu at (257.4, 170.0)
- added Q4: MMBT2222, SOT23, F.Cu at (275.4, 173.0)
- added Q5: BD139-16, SOT32_TO126, F.Cu at (273.2, 181.8)
- added Q6: MMBT2222, SOT23, F.Cu at (243.7, 180.4)
- added R1: 51R, RES_0603, F.Cu at (250.8, 188.4)
- added R10: 1k, RES_0603, F.Cu at (268.0, 177.4)
- added R11: 0.1R, RES_0805, F.Cu at (273.2, 176.6)
- added R12: 20k, RES_0603, F.Cu at (263.8, 205.2)
- added R13: 12k, RES_0603, F.Cu at (262.0, 199.4)
- added R14: 20R, RES_0603, F.Cu at (247.0, 181.2)
- added R2: 1k, RES_0603, F.Cu at (272.8, 173.2)
- added R3: 220R, RES_0603, F.Cu at (256.2, 197.0)
- added R4: 51R, RES_0603, F.Cu at (250.8, 186.4)
- added R5: 30k, RES_0603, F.Cu at (268.0, 175.6)
- added R6: 51R, RES_0603, F.Cu at (250.8, 190.4)
- added R7: 100, RES_0603, F.Cu at (255.7, 165.2)
- added R8: 20R, RES_0603, F.Cu at (247.0, 179.3)
- added R9: 1k, RES_0603, F.Cu at (241.1, 180.6)
- added TP1: TESTPOINT, TESTPOINT_1MM, F.Cu at (265.6, 175.6)
- added TP2: TESTPOINT, TESTPOINT_1MM, F.Cu at (275.6, 184.0)
- added XL1: CONN_2, CONN_MF2_MRB, F.Cu at (272.0, 194.0)
- added XL5: CONN_3, SIL-3, F.Cu at (236.2, 187.2)
- added XL6: ST_SWD, SIL-4, F.Cu at (236.2, 197.0)
- added XL7: CONN_1, SIL-1, F.Cu at (247.2, 190.2)
- added XTAL2: 12.0MHz, CRYSTAL_0503x4-4, F.Cu at (259.0, 198.3)
Routing:
- net GND: track 0.00 -> 454.6 mm, vias 0 -> 54
- net +3.3V: track 0.00 -> 91.2 mm, vias 0 -> 6
- net +BATT: track 0.00 -> 78.7 mm, vias 0 -> 1
- net /Buzzer: track 0.00 -> 39.6 mm, vias 0 -> 2
- net /XotarIn: track 0.00 -> 34.4 mm, vias 0 -> 1
- net /XotarPower: track 0.00 -> 29.8 mm, vias 0 -> 2
- net /DAC: track 0.00 -> 28.2 mm, vias 0 -> 2
- net /LED3_OUT: track 0.00 -> 16.9 mm
- net /TIM: track 0.00 -> 16.6 mm
- net /LED1_OUT: track 0.00 -> 13.8 mm, vias 0 -> 1
- net /TX1: track 0.00 -> 13.1 mm
- net /LED2_OUT: track 0.00 -> 12.8 mm
- net /LED4_OUT: track 0.00 -> 12.8 mm
- net N-0000039: track 0.00 -> 12.2 mm
- net /RX1: track 0.00 -> 11.5 mm
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- added copper zone on B.Cu, net GND
- added copper zone on F.Cu, net GND
Other:
- board outline added: 45 x 45 mm
