File: SciFi/IrGirandole/Girandole_hw/girandole.sch (KiCad schematic (older format))
At the start: 52 parts

Commit message: 
Parts:
- removed C?: 1000pF, symbol C
- removed D? (x3): LED, symbol LED
- removed DA?: LP2951, symbol LP2951
- removed Q?: MMBT2222, symbol NPN
- removed R?: 120k, symbol R
- removed R?: 200k, symbol R
- removed R?: 1k, symbol R
- added C3: 1000u, symbol CP
- added C4: 10u, CAP_0805, symbol C
- added C5: 0.1u, CAP_0603, symbol C
- added D2, D3, D7: LED, symbol LED
- added DA1, DA2, DA3, DA4: LM317_SO8, symbol LM317_SO8
- added F1, F3, F4, F5: FUSE0R, symbol FUSE0R
- added Q5, Q?: IRLML9303, symbol IRLML6302
- added R14, R17, R19, R8: 5R1*, RES_1206, symbol R
- added R15, R18, R20, R9: 22R*, RES_1206, symbol R
- added R16: 100k, RES_0603, symbol R
- DD1: renamed from DD?; value EEPROM_I2C -> AT24C02
- gave numbers to parts that had none: 27
Connections:
- net labels added: LED1_INTER, LED1_OUT, LED2_INTER, LED2_OUT, LED3_INTER, LED3_OUT, LED4_INTER, LED4_OUT, LED_IN
- net labels removed: +BATT
- wire segments 154 -> 208
- no-connect marks 17 -> 14
Other:
- moved on the sheet: BZ1, C1, C15, C18, C2, C38, C39, C40, C41, C43, C44, D1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

Commit message: 
Parts:
- removed C1: 0.1u, CAP_0402, symbol C
- removed C6: 1000u, symbol CP
- removed C7: 0.1u, symbol C
- removed C8: 10u, symbol C
- removed C9: 1u, symbol C
- removed D1, D2, D3, D7: LED, symbol LED
- removed D4, D5, D6: SS14, symbol D_SHOTTKY
- removed DA1, DA2, DA3, DA4: LM317_SO8, symbol LM317_SO8
- removed DD1: AT24C02, symbol EEPROM_I2C
- removed F1, F2, F3, F4, F5: FUSE0R, symbol FUSE0R
- removed Q5, Q?: IRLML9303, symbol IRLML6302
- removed R10, R11: 22, RES_0603, symbol R
- removed R12: 1k5, RES_0603, symbol R
- removed R14, R17, R19, R8: 5R1*, RES_1206, symbol R
- removed R15, R18, R20, R9: 22R*, RES_1206, symbol R
- removed R16: 100k, RES_0603, symbol R
- removed R2, R5: 4k7, RES_0603, symbol R
- removed XL1: USB_MINI_B, symbol USB_MINI_B
- removed XL2, XL3: CONN_1, symbol CONN_1
- removed XL4: BARREL_SOCKET, symbol BARREL_SOCKET
- added C? (x2): 1n, CAP_0603, symbol C
- added C? (x2): 1u, CAP_0603, symbol C
- added C?: 10u, CAP_0805, symbol C
- added C?: 3.3pF, CAP_0603, symbol C
- added D? (x4): LED, symbol LED
- added DA?: LP2951, ~, symbol LP2951
- added DA?: MAX4453, symbol GENERIC_8PIN
- added F? (x7): FUSE0R, symbol FUSE0R
- added Q? (x2): MMBT2222, symbol NPN
- added Q?: BD139-16, symbol NPN
- added R?: 20k, RES_0603, symbol R
- added R?: 12k, RES_0603, symbol R
- added R? (x3): 1k, RES_0603, symbol R
- added R?: 20R, RES_0603, symbol R
- added R?: 0.1R, RES_0805, symbol R
- added R?: 30k, RES_0603, symbol R
- added TP? (x2): TESTPOINT, symbol TESTPOINT
- added XL?: CONN_2, symbol CONN_2
Connections:
- net labels added: +BATT, CURR_SNS, DAC, ONE_LED, TIM
- net labels removed: +5V, LED1_INTER, LED2_INTER, LED3_INTER, LED4_INTER, LED4_OUT, LED_IN, PWR_IN_BAT, PWR_IN_EXT, SCL, SDA, USB_CABLE, USB_DM, USB_DP, VCC, XotarLED
- wire segments 208 -> 175
- no-connect marks 14 -> 18
Other:
- note added: "3xAAA\nor\n12V"
- note added: "Address\nsettings"
- note added: "Peripherals usage\n\nUSB\nUART1 - output/input\nTIM1 Ch1 - Xotar LED\nTIM2 Ch2,3,4 - RGB LED\nTIM3 Ch1 - Xotar In\nTIM15 Ch1 - Buzzer\nTIM ? - Xotar Data timings\n"
- note added: "Stabilizer"
- note removed: "+BATTERY"
- note removed: "-BATTERY"
- note removed: "Peripherals usage\n\nUSB\nUART1 - output/input\nTIM1 Ch1 - Xotar LED\nTIM2 Ch2,3,4 - RGB LED\nTIM3 Ch1 - Xotar In\nTIM4 Ch3 (TIM16C1) - Buzzer\nTIM ? - Xotar Data timings\n"
- note removed: "USB"
- moved on the sheet: BZ1, C3, C4, C5

Commit message: Girandole hw completed
Parts:
- removed C4: 10u, CAP_0805, symbol C
- removed Q?: BD139-16, symbol NPN
- added C11: 0.1u, CAP_0603, symbol C
- added D1: LED, ~, symbol LED
- added F8: FUSE0R, symbol FUSE0R
- added HOLE1, HOLE2, HOLE3, HOLE4: HOLE_METALLED, symbol HOLE_METALLED
- added Q5: BD139-16, symbol NPN_B1C2E3
- added R14: 20R, RES_0603, symbol R
- gave numbers to parts that had none: 32
Connections:
- net labels added: LED4_OUT
- net labels removed: ONE_LED
- wire segments 175 -> 187
Other:
- moved on the sheet: BZ1, C15, C18, C2, C38, C39, C40, C41, C43, C44, DD2, Q1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

Commit message: Sch: 10uF added, 30k creplaced with 20k. Soft: DAC values adjusted
Parts:
- added C_AddItSomehow: 10uF, CAP_0603, symbol C
- C1: value 3.3pF -> DoNotMount
- R5: value 30k -> 20k
Connections:
- wire segments 187 -> 188
Changed lines of the file:
@@
-EESchema Schematic File Version 2  date 03/07/2013 13:12:06
+EESchema Schematic File Version 2  date 11/07/2013 14:06:46
 LIBS:Connectors_kl
 LIBS:pcb_details
@@
 Sheet 1 1
 Title ""
-Date "3 jul 2013"
+Date "11 jul 2013"
 Rev ""
 Comp ""
@@
 	0    -1   -1   0
 $EndComp
-Text Label 13200 7550 0    61   ~ 0
+Text Label 12650 7550 0    61   ~ 0
 DAC
 $Comp
@@
 P 13450 7850
 F 0 "R5" V 13530 7700 50  0000 C CNN
-F 1 "30k" V 13450 7850 50  0000 C CNN
+F 1 "20k" V 13450 7850 50  0000 C CNN
 F 2 "RES_0603" V 13530 7950 28  0000 C CNN
 F 3 "" H 13450 7850 60  0000 C CNN
@@
 P 14450 7550
 F 0 "C1" V 14650 7750 50  0000 L CNN
-F 1 "3.3pF" V 14550 7650 50  0000 L CNN
+F 1 "DoNotMount" V 14550 7650 50  0000 L CNN
 F 2 "CAP_0603" V 14550 7400 28  0000 C BNN
 F 3 "~" H 14450 7550 60  0000 C CNN
@@
 Connection ~ 1800 9600
 Wire Wire Line
-	13450 7550 13200 7550
+	12900 7550 12650 7550
 Wire Wire Line
 	8350 8450 8650 8450
@@
 	14800 7000 15200 7000
 Connection ~ 15200 7000
+$Comp
+L C C_AddItSomehow
+U 1 1 51DE8695
+P 13100 7550
+F 0 "C_AddItSomehow" V 13300 7450 50  0000 L CNN
+F 1 "10uF" V 13200 7650 50  0000 L CNN
+F 2 "CAP_0603" V 13200 7400 28  0000 C BNN
+F 3 "~" H 13100 7550 60  0000 C CNN
+	1    13100 7550
+	0    -1   -1   0
+$EndComp
+Wire Wire Line
+	13300 7550 13450 7550
 $EndSCHEMATC
