File: Calmari/WitcherLocket/WitcherLocket_hw/WitcherLocket.sch (KiCad schematic (older format))
At the start: 25 parts, among them SW1 SWITCH_2X, SW2 SWITCH_2X, SW3 SWITCH_2X, SW4 SWITCH_2X

Commit message: 
Parts:
- added HOLE1, HOLE2, HOLE3, HOLE4: HOLE_METALLED, symbol HOLE_METALLED
Connections:
- wire segments 64 -> 69
Changed lines of the file:
@@
-EESchema Schematic File Version 2  date 23/03/2013 22:32:17
+EESchema Schematic File Version 2  date 24/05/2013 18:50:32
 LIBS:Connectors_kl
 LIBS:pcb_details
@@
 LIBS:st_kl
 LIBS:Transistors_kl
+LIBS:WitcherLocket-cache
 EELAYER 27 0
 EELAYER END
@@
 Sheet 1 1
 Title ""
-Date "23 mar 2013"
+Date "24 may 2013"
 Rev ""
 Comp ""
@@
 	9600 4650 9600 5100
 Connection ~ 9600 5100
+Wire Wire Line
+	2500 1550 2500 2700
+Connection ~ 2500 2550
+Wire Wire Line
+	2500 2550 2400 2550
+Wire Wire Line
+	2500 2250 2400 2250
+$Comp
+L GND #PWR023
+U 1 1 519F79EF
+P 2500 2700
+F 0 "#PWR023" H 2590 2680 30  0001 C CNN
+F 1 "GND" H 2500 2620 30  0001 C CNN
+F 2 "" H 2500 2700 60  0001 C CNN
+F 3 "" H 2500 2700 60  0001 C CNN
+	1    2500 2700
+	1    0    0    -1
+$EndComp
+$Comp
+L HOLE_METALLED HOLE4
+U 1 1 519F79F5
+P 2100 2550
+F 0 "HOLE4" H 1600 2500 60  0000 C CNN
+F 1 "HOLE_METALLED" H 1550 2600 60  0000 C CNN
+F 2 "" H 2100 2550 60  0001 C CNN
+F 3 "" H 2100 2550 60  0001 C CNN
+	1    2100 2550
+	1    0    0    -1
+$EndComp
+$Comp
+L HOLE_METALLED HOLE3
+U 1 1 519F79FB
+P 2100 2250
+F 0 "HOLE3" H 1600 2200 60  0000 C CNN
+F 1 "HOLE_METALLED" H 1550 2300 60  0000 C CNN
+F 2 "" H 2100 2250 60  0001 C CNN
+F 3 "" H 2100 2250 60  0001 C CNN
+	1    2100 2250
+	1    0    0    -1
+$EndComp
+$Comp
+L HOLE_METALLED HOLE2
+U 1 1 519F7A03
+P 2100 1900
+F 0 "HOLE2" H 1600 1850 60  0000 C CNN
+F 1 "HOLE_METALLED" H 1550 1950 60  0000 C CNN
+F 2 "" H 2100 1900 60  0000 C CNN
+F 3 "" H 2100 1900 60  0000 C CNN
+	1    2100 1900
+	1    0    0    -1
+$EndComp
+$Comp
+L HOLE_METALLED HOLE1
+U 1 1 519F7A12
+P 2100 1550
+F 0 "HOLE1" H 1600 1500 60  0000 C CNN
+F 1 "HOLE_METALLED" H 1550 1600 60  0000 C CNN
+F 2 "" H 2100 1550 60  0000 C CNN
+F 3 "" H 2100 1550 60  0000 C CNN
+	1    2100 1550
+	1    0    0    -1
+$EndComp
+Wire Wire Line
+	2400 1550 2500 1550
+Connection ~ 2500 2250
+Wire Wire Line
+	2400 1900 2500 1900
+Connection ~ 2500 1900
 $EndSCHEMATC

Commit message: 
Parts:
- added HOLE5, HOLE6: HOLE_METALLED, symbol HOLE_METALLED
Connections:
- wire segments 69 -> 64
- no-connect marks 8 -> 14
Other:
- moved on the sheet: C1, C2, C3, C4, DA1, L1, XL1, XL2

Commit message: led resistors change
Parts:
- R1, R3: value 47R -> 51R
- R2, R4: value 47R -> 10R
Changed lines of the file:
@@
-EESchema Schematic File Version 2  date 29/05/2013 23:55:25
+EESchema Schematic File Version 2  date 10/07/2013 19:59:24
 LIBS:Connectors_kl
 LIBS:pcb_details
@@
 Sheet 1 1
 Title ""
-Date "28 may 2013"
+Date "10 jul 2013"
 Rev ""
 Comp ""
@@
 P 8250 2050
 F 0 "R1" V 8330 1900 50  0000 C CNN
-F 1 "47R" V 8250 2050 50  0000 C CNN
+F 1 "51R" V 8250 2050 50  0000 C CNN
 F 2 "RES_0603" V 8330 2150 28  0000 C CNN
 F 3 "" H 8250 2050 60  0000 C CNN
@@
 P 8250 3000
 F 0 "R2" V 8330 2850 50  0000 C CNN
-F 1 "47R" V 8250 3000 50  0000 C CNN
+F 1 "10R" V 8250 3000 50  0000 C CNN
 F 2 "RES_0603" V 8330 3100 28  0000 C CNN
 F 3 "" H 8250 3000 60  0000 C CNN
@@
 P 8250 4000
 F 0 "R3" V 8330 3850 50  0000 C CNN
-F 1 "47R" V 8250 4000 50  0000 C CNN
+F 1 "51R" V 8250 4000 50  0000 C CNN
 F 2 "RES_0603" V 8330 4100 28  0000 C CNN
 F 3 "" H 8250 4000 60  0000 C CNN
@@
 P 8250 5100
 F 0 "R4" V 8330 4950 50  0000 C CNN
-F 1 "47R" V 8250 5100 50  0000 C CNN
+F 1 "10R" V 8250 5100 50  0000 C CNN
 F 2 "RES_0603" V 8330 5200 28  0000 C CNN
 F 3 "" H 8250 5100 60  0000 C CNN
