File: Calmari/Torches/Torch3/Torch3_hw/torch3.sch (KiCad schematic (older format))
At the start: 42 parts

Commit message: Mushrooms added
Other:
- note added: "If just a button needed (no touch) - \nremove touch sensor and solder the fuse"
Changed lines of the file:
@@
-EESchema Schematic File Version 2  date 18/02/2013 02:16:01
+EESchema Schematic File Version 2  date 28/02/2013 18:07:00
 LIBS:Connectors_kl
 LIBS:pcb_details
@@
 Sheet 1 1
 Title ""
-Date "17 feb 2013"
+Date "28 feb 2013"
 Rev ""
 Comp ""
@@
 Comment4 ""
 $EndDescr
+Text Notes 2550 1600 0    60   ~ 0
+If just a button needed (no touch) - \nremove touch sensor and solder the fuse
 Connection ~ 4100 6350
 Wire Wire Line
