File: Modules/Rinca/Rinca_hw/Rinca.kicad_pcb (KiCad board)
At the start: 2 copper layers, 49 x 66 mm, 69 parts, among them SW1 SWITCH, SW2 BUTTON, SW3 BUTTON, SW4 BUTTON

Commit message: Quetta added
Routing:
- net GND: track 550.4 -> 552.8 mm, vias 96 -> 99
- net +3.3V: track 218.8 -> 217.2 mm
- net /GPIO1: track 37.1 -> 36.2 mm
- net /Ch1_ERROR: track 40.3 -> 40.9 mm
Other:
- net class Default: clearance 0.20066 -> 0.2; trace_width 0.20066 -> 0.2; via_dia 1.00076 -> 0.9; via_drill 0.50038 -> 0.4
- net class Wide: clearance 0.20066 -> 0.2; trace_width 0.50038 -> 0.5; via_dia 1.00076 -> 0.9; via_drill 0.50038 -> 0.4
- rule trace_clearance: 0.20066 -> 0.2
