File: HandyDevices/BrainEnchanter/Hardware/BrainEnch.kicad_pcb (KiCad board)
At the start: 2 copper layers, 50 x 57 mm, 57 parts, among them Q1 MMBT2222, Q2 MMBT2222, SW1 BUTTON, SW2 BUTTON, SW3 BUTTON, SW4 BUTTON, SW5 BUTTON

Commit message: BrainEnch PCB ready for production
Parts:
- added L3: 10uH, IND_0805, B.Cu at (184.2, 178.0)
- added TP3: TESTPOINT, TESTPOINT_1MM, B.Cu at (186.8, 165.2)
- Q2: value MMBT2222 -> NPN
- R5: value 1.94k -> 81k
- R6: value 1k -> 10k
- XTAL1: footprint CRYSTAL_KX26 -> CRYSTAL_KX26_NOGND
- moved R4 41.8 mm to (202.8, 157.8), turned to 270 degrees
- moved R1 22.9 mm to (174.6, 159.8), turned to 90 degrees
- moved R3 15.9 mm to (173.2, 168.8), turned to 180 degrees
- moved R9 10.6 mm to (197.0, 165.4)
- moved R8 10.4 mm to (197.0, 163.6), turned to 180 degrees
- moved C15 10.2 mm to (180.2, 162.0), turned to 270 degrees
- moved R2 8.41 mm to (183.8, 184.2)
- moved R5 8.33 mm to (183.8, 162.0), turned to 270 degrees
- moved C11 8.32 mm to (180.6, 187.6)
- moved C5 8.21 mm to (184.6, 180.0)
- moved C4 8.10 mm to (188.4, 190.2)
- moved C2 8.02 mm to (195.0, 175.8)
- moved C3 7.96 mm to (199.0, 185.8)
- moved DD1 7.96 mm to (191.8, 183.0)
- moved C6 7.96 mm to (184.6, 181.8)
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Connections:
- C11 pad 1: N-0000041 -> N-0000038
- C5 pad 1: +3.3V -> N-000004
- C6 pad 1: +3.3V -> N-000004
- C9 pad 1: N-0000042 -> N-0000037
- DD1 pad 1: (no net) -> +3.3V
- DD1 pad 3: N-0000041 -> N-0000038
- DD1 pad 9: +3.3V -> N-000004
- Q2 pad 2: /BRAIN_C -> /CURR_SNS
- Q2 pad 3: /CURR_SNS -> /BRAIN_C
- R2 pad 2: N-0000042 -> N-0000037
- XTAL1 pad 1: N-0000041 -> N-0000037
- XTAL1 pad 2: N-0000042 -> N-0000038
Routing:
- net GND: track 0.00 -> 606.9 mm, vias 0 -> 70
- net +3.3V: track 0.00 -> 147.0 mm, vias 0 -> 6
- net /Buzzer: track 0.00 -> 46.6 mm, vias 0 -> 2
- net +BATT: track 0.00 -> 44.4 mm, vias 0 -> 1
- net /BTN3: track 0.00 -> 39.2 mm, vias 0 -> 1
- net /LCD_SCLK: track 0.00 -> 35.2 mm, vias 0 -> 1
- net /BTN1: track 0.00 -> 33.9 mm, vias 0 -> 1
- net /BTN4: track 0.00 -> 33.5 mm, vias 0 -> 1
- net /LCD_XCS: track 0.00 -> 32.4 mm, vias 0 -> 1
- net /UART_RX: track 0.00 -> 32.2 mm
- net /LCD_SDA: track 0.00 -> 30.2 mm, vias 0 -> 1
- net /LCD_XRES: track 0.00 -> 28.8 mm, vias 0 -> 1
- net /UART_TX: track 0.00 -> 28.3 mm
- net /BTN5: track 0.00 -> 27.9 mm, vias 0 -> 1
- net /BTN2: track 0.00 -> 25.3 mm, vias 0 -> 1
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- added copper zone on B.Cu, net GND
- added copper zone on F.Cu, net GND
