File: Calmari/Calma04/Calma04_hw/Calma04.sch (KiCad schematic (older format))
At the start: 36 parts, among them Q1 ALS-PT19-315C, SW1 SWITCH, SW2 BUTTON

Commit message: calma04 pcb added
Parts:
- removed HOLE1: HOLE_METALLED, symbol HOLE_METALLED
- added C14, C15: 10u, symbol C
- added DA3: MCP73832, symbol MCP73832
- added R4: 2k, symbol R
- added XL10, XL11, XL12, XL13, XL8, XL9: CONN_1, symbol CONN_1
- added XL7: USB_MICRO_B, symbol USB_MINI_B
Connections:
- net labels added: +5V, Charge
- wire segments 101 -> 126
- no-connect marks 30 -> 31
Other:
- note added: "Connectors for spliting pcb"
- note added: "Li-Ion charger\n2k => 0.5 A"
- note added: "USB"
- moved on the sheet: C1, C10, C11, C12, C13, C2, C3, C4, C5, C6, C7, C8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

Commit message: 
Parts:
- added R6: 10k, RES_0603, symbol R
- added R7: 120k, RES_0603, symbol R
Connections:
- net labels added: FB
- wire segments 126 -> 128
- no-connect marks 31 -> 30
Other:
- moved on the sheet: R3
Changed lines of the file:
@@
-EESchema Schematic File Version 2  date 14/07/2013 23:49:17
+EESchema Schematic File Version 2  date 16/07/2013 00:07:37
 LIBS:Connectors_kl
 LIBS:pcb_details
@@
 Sheet 1 1
 Title ""
-Date "14 jul 2013"
+Date "15 jul 2013"
 Rev ""
 Comp ""
@@
 L R R3
 U 1 1 51E13D2B
-P 9300 2800
-F 0 "R3" V 9380 2650 50  0000 C CNN
-F 1 "13R" V 9300 2800 50  0000 C CNN
-F 2 "RES_0603" V 9380 2900 28  0000 C CNN
-F 3 "~" H 9300 2800 60  0000 C CNN
-	1    9300 2800
+P 9950 3100
+F 0 "R3" V 10030 2950 50  0000 C CNN
+F 1 "13R" V 9950 3100 50  0000 C CNN
+F 2 "RES_0603" V 10030 3200 28  0000 C CNN
+F 3 "~" H 9950 3100 60  0000 C CNN
+	1    9950 3100
 	1    0    0    -1
 $EndComp
@@
 L GND #PWR035
 U 1 1 51E13D38
-P 9300 3150
-F 0 "#PWR035" H 9390 3130 30  0001 C CNN
-F 1 "GND" H 9300 3070 30  0001 C CNN
-F 2 "" H 9300 3150 60  0001 C CNN
-F 3 "" H 9300 3150 60  0001 C CNN
-	1    9300 3150
+P 9950 3450
+F 0 "#PWR035" H 10040 3430 30  0001 C CNN
+F 1 "GND" H 9950 3370 30  0001 C CNN
+F 2 "" H 9950 3450 60  0001 C CNN
+F 3 "" H 9950 3450 60  0001 C CNN
+	1    9950 3450
 	1    0    0    -1
 $EndComp
@@
 NoConn ~ 5750 2750
 NoConn ~ 5750 2650
-NoConn ~ 5750 2550
 NoConn ~ 5750 2450
 NoConn ~ 5750 2350
@@
 	1    0    0    -1
 $EndComp
-Text Notes 9500 2800 0    60   ~ 0
+Text Notes 10100 3200 0    60   ~ 0
 R=252/Iled[mA]
 $Comp
@@
 	8800 2750 8800 2850
 Wire Wire Line
-	9300 3050 9300 3150
-Wire Wire Line
-	9200 2450 9300 2450
-Wire Wire Line
-	9300 2350 9300 2550
-Wire Wire Line
-	9200 2350 9300 2350
-Connection ~ 9300 2450
+	9950 3350 9950 3450
 Wire Wire Line
 	8100 1950 8100 1500
@@
 Text Notes 12750 3150 0    60   ~ 0
 Connectors for spliting pcb
+$Comp
+L R R6
+U 1 1 51E42641
+P 9600 2600
+F 0 "R6" V 9680 2450 50  0000 C CNN
+F 1 "10k" V 9600 2600 50  0000 C CNN
+F 2 "RES_0603" V 9680 2700 28  0000 C CNN
+F 3 "~" H 9600 2600 60  0000 C CNN
+	1    9600 2600
+	-1   0    0    1
+$EndComp
+$Comp
+L R R7
+U 1 1 51E42797
+P 10200 2350
+F 0 "R7" V 10280 2200 50  0000 C CNN
+F 1 "120k" V 10200 2350 50  0000 C CNN
+F 2 "RES_0603" V 10280 2450 28  0000 C CNN
+F 3 "~" H 10200 2350 60  0000 C CNN
+	1    10200 2350
+	0    -1   -1   0
+$EndComp
+Wire Wire Line
+	9200 2350 9950 2350
+Wire Wire Line
+	9200 2450 9200 2850
+Wire Wire Line
+	9200 2850 9950 2850
+Connection ~ 9600 2350
+Wire Wire Line
+	10450 2350 10750 2350
+Connection ~ 9600 2850
+Wire Wire Line
+	5750 2550 6000 2550
+Text Label 6000 2550 0    60   ~ 0
+FB
+Text Label 10750 2350 2    60   ~ 0
+FB
 $EndSCHEMATC

Commit message: 
Connections:
- wire segments 128 -> 130
Other:
- moved on the sheet: R3, R6

Commit message: + Calma04
Parts:
- added R?: 2k, symbol R
Connections:
- wire segments 130 -> 131
Other:
- note added: "Place resistor\nsomehow if \nLED Off during\npower-up is \nrequired"
Changed lines of the file:
@@
-EESchema Schematic File Version 2  date 22/07/2013 12:11:27
+EESchema Schematic File Version 2
 LIBS:Connectors_kl
 LIBS:pcb_details
@@
 Sheet 1 1
 Title ""
-Date "22 jul 2013"
+Date "26 jan 2014"
 Rev ""
 Comp ""
@@
 	8600 2750 8600 2850
 Wire Wire Line
-	8200 2600 8200 2300
+	8200 2300 8200 2700
 Wire Wire Line
 	6500 2600 8200 2600
@@
 	5000 8500 5000 8550
 Connection ~ 5000 8500
+$Comp
+L GND #PWR?
+U 1 1 52E4EA42
+P 8200 3300
+F 0 "#PWR?" H 8290 3280 30  0001 C CNN
+F 1 "GND" H 8200 3220 30  0001 C CNN
+F 2 "" H 8200 3300 60  0001 C CNN
+F 3 "" H 8200 3300 60  0001 C CNN
+	1    8200 3300
+	1    0    0    -1
+$EndComp
+$Comp
+L R R?
+U 1 1 52E4EA48
+P 8200 2950
+F 0 "R?" V 8280 2950 50  0000 C CNN
+F 1 "2k" V 8200 2950 50  0000 C CNN
+F 2 "" H 8200 2950 60  0001 C CNN
+F 3 "" H 8200 2950 60  0001 C CNN
+	1    8200 2950
+	1    0    0    -1
+$EndComp
+Wire Wire Line
+	8200 3200 8200 3300
+Connection ~ 8200 2600
+Text Notes 7450 2850 0    60   ~ 0
+Place resistor\nsomehow if \nLED Off during\npower-up is \nrequired
 $EndSCHEMATC
