File: Calmari/Mushrooms/Mushroom_hw/mushroom.sch (KiCad schematic (older format))
At the start: 40 parts

Commit message: NCP5007 added
Parts:
- removed ANT1: ANT_PCB_MONO, ~, symbol ANT_PCB_MONO
- removed C10, C9: 10pF, CAP_0402, symbol C
- removed C11, C21, C23, C4, C5, C7: 0.1u, symbol C
- removed C22, C24: 10u, symbol C
- removed C3, C6, C8: 220pF, symbol C
- removed D2: BAT54WS, symbol D_SHOTTKY
- removed DA1: NCP1400, symbol NCP1400
- removed DD?: CC2500, ~, symbol CC2500
- removed L2: 22uH, symbol L
- removed R10, R8, R9: 51R, RES_0603, symbol R
- removed R2: 56k, symbol R
- removed XTAL1: 27MHz, 03225, symbol CRYSTAL_H
- added ANT?: ANT_GENERAL, symbol ANT_GENERAL
- added C? (x6): 0.1u, symbol C
- added C? (x2): 10u, symbol C
- added C? (x3): 220pF, symbol C
- added C? (x2): 10pF, CAP_0402, symbol C
- added C? (x2): 100pF, CAP_0402, symbol C
- added C? (x2): 1pF, CAP_0402, symbol C
- added C?: 1.8pF, CAP_0402, symbol C
- added C?: 1.5pF, CAP_0402, symbol C
- added C?: 4.7u, CAP_0603, symbol C
- added C?: 1u, CAP_0603, symbol C
- added D?: D_SHOTTKY, ~, symbol D_SHOTTKY
- added DA?: NCP583SQ, ~, symbol NCP583SQ
- added DA?: NCP5007, symbol NCP5007
- added DD?: CC2500, symbol CC2500
- added F?: FUSE0R, symbol FUSE0R
- added L? (x3): 1.2nH, IND_0402, symbol L
- added L?: 22uH, IND_0402, symbol L
- added R?: 56k, symbol R
- added R? (x2): 330k, RES_0603, symbol R
- added R?: R, RES_0603, symbol R
- added SW?: SWITCH, symbol SWITCH
- added XTAL?: 27MHz, 03225, symbol CRYSTAL_H
Connections:
- net labels added: Ant1, Ant2, BAT_IN
- net labels removed: Lout, RF1, RF2
- wire segments 115 -> 157
- no-connect marks 16 -> 17
Other:
- note added: "Battery\nmeasurement"
- note added: "UART"
- note removed: "Debug port"
- note removed: "Indication"
- note removed: "Matching circuit"
- note removed: "Radio"
- moved on the sheet: B1, B?, C12, C13, C14, C15, C16, C18, TP1, TP2, XL1, XL2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

Commit message: TPS61042 added
Parts:
- removed C?: 4.7u, CAP_0603, symbol C
- removed C?: 1u, CAP_0603, symbol C
- removed D?: D_SHOTTKY, ~, symbol D_SHOTTKY
- removed DA?: NCP5007, symbol NCP5007
- removed L?: 22uH, IND_0402, symbol L
- removed R?: R, RES_0603, symbol R
- added C?: 0.1u, symbol C
- added C? (x2): 10u, symbol C
- added D?: SS14, ~, symbol D_SHOTTKY
- added DA?: TPS61042, symbol TPS61042
- added L?: 6.8uH, IND_1210, symbol L
- added Q? (x5): LED_RGB, ~, symbol LED_RGB
- added R?: 13R, RES_0603, symbol R
- added R?: 10k, RES_0603, symbol R
- added R?: 120k, RES_0603, symbol R
- added R?: 100k, symbol R
Connections:
- net labels added: BLUE_PWM, BRIGHTNESS, GREEN_PWM, RED_N, RED_P, RED_PWM
- net labels removed: BLUE_LED, GREEN_LED, RED_LED
- wire segments 157 -> 183
- no-connect marks 17 -> 16
Other:
- note added: "Choose capacitor \nmax voltage carefully\n(30v recommended)"
- note added: "R=252/Iled[mA]"

Commit message: Sch completed
Parts:
- removed ANT?: ANT_GENERAL, symbol ANT_GENERAL
- removed C? (x2): 100pF, CAP_0402, symbol C
- removed C? (x2): 1pF, CAP_0402, symbol C
- removed C?: 1.8pF, CAP_0402, symbol C
- removed C?: 1.5pF, CAP_0402, symbol C
- removed F?: FUSE0R, symbol FUSE0R
- removed L? (x3): 1.2nH, IND_0402, symbol L
- removed Q? (x2): LED_RGB, ~, symbol LED_RGB
- added ANT1: ANT_PCB_NOCNTR, ~, symbol ANT_PCB_NOCNTR
- added C14, C20: 0.1u, symbol C
- added C15, C16, C21, C30: 10u, symbol C
- added C22, C28, C31: 0.1u, CAP_0603, symbol C
- added D2, D3: SS14, ~, symbol D_SHOTTKY
- added DA3, DA4: TPS61042, symbol TPS61042
- added F1, F2, F3, F4, F5, F6, F7, F8, F9: FUSE0R, ~, symbol FUSE0R
- added L2, L3: 6.8uH, IND_1210, symbol L
- added Q1, Q4, Q6: LED_RGB_WS2812B, ~, symbol LED_RGB_WS2812B
- added R10, R15: 120k, RES_0603, symbol R
- added R12, R5: 100k, symbol R
- added R13, R8: 10k, RES_0603, symbol R
- added R14, R9: 13R, RES_0603, symbol R
- added TP1: TESTPOINT, symbol TESTPOINT
- added XL10, XL11, XL12, XL15, XL16, XL17, XL20, XL21, XL22, XL25, XL26, XL27, XL5, XL6, XL7: CONN_2, ~, symbol CONN_2
- added XL13, XL18, XL23, XL28, XL8: CONN_1, ~, symbol CONN_1
- added XL14, XL19, XL24, XL4, XL9: CONN_3, ~, symbol CONN_3
- C10: renamed from C16; footprint CAP_0402 -> CAP_0603
- C17, C18: renamed from C?; footprint CAP_0402 -> CAP_0603
- C4: renamed from C13; footprint CAP_0402 -> CAP_0603
- C5: renamed from C18; footprint CAP_0402 -> CAP_0603
- C7: renamed from C14; footprint CAP_0402 -> CAP_0603
- C9: renamed from C15; footprint CAP_0402 -> CAP_0603
- gave numbers to parts that had none: 33
- renumbered C12 to C3, TP1 to TP2, TP2 to TP3, XL2 to XL1, XL1 to XL2
Connections:
- net labels added: Ant, BLUE_N, BLUE_P, DIN0, DIN1, DIN2, DIN3, DIN4, GREEN_N, GREEN_P
- net labels removed: Ant1, Ant2
- wire segments 183 -> 293
- no-connect marks 16 -> 21
Other:
- moved on the sheet: B1, B2, B3, C1, C11, C12, C13, C17, C18, C19, C2, C23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

Commit message: LedPcb completed and added
Parts:
- removed SW1: SWITCH, symbol SWITCH
- added SW?: SWITCH_H, ~, symbol SWITCH_H
Connections:
- wire segments 293 -> 294
Changed lines of the file:
@@
 Sheet 1 1
 Title ""
-Date "20 mar 2014"
+Date "22 mar 2014"
 Rev ""
 Comp ""
@@
 	1    0    0    -1
 $EndComp
-$Comp
-L SWITCH SW1
-U 1 1 53285EAC
-P 2900 9900
-F 0 "SW1" H 2650 10150 60  0000 C CNN
-F 1 "SWITCH" H 3000 10150 60  0000 C CNN
-F 2 "" H 2900 9900 60  0000 C CNN
-F 3 "" H 2900 9900 60  0000 C CNN
-	1    2900 9900
-	-1   0    0    -1
-$EndComp
 NoConn ~ 2650 9800
 Text Label 2200 9900 0    60   ~ 0
@@
 NoConn ~ 7250 3250
 NoConn ~ 7250 3350
+$Comp
+L SWITCH_H SW?
+U 1 1 532DDC0D
+P 2900 9900
+F 0 "SW?" H 2650 10150 60  0000 C CNN
+F 1 "SWITCH_H" H 3000 10150 60  0000 C CNN
+F 2 "~" H 2900 9900 60  0000 C CNN
+F 3 "~" H 2900 9900 60  0000 C CNN
+	1    2900 9900
+	-1   0    0    -1
+$EndComp
+$Comp
+L GND #PWR?
+U 1 1 532DDC29
+P 2950 10200
+F 0 "#PWR?" H 3040 10180 30  0001 C CNN
+F 1 "GND" H 2950 10120 30  0001 C CNN
+F 2 "" H 2950 10200 60  0001 C CNN
+F 3 "" H 2950 10200 60  0001 C CNN
+	1    2950 10200
+	1    0    0    -1
+$EndComp
+Wire Wire Line
+	2950 10100 2950 10200
 $EndSCHEMATC

Commit message: 
Parts:
- removed XL10, XL11, XL12, XL15, XL16, XL17, XL20, XL21, XL22, XL25, XL26, XL27, XL5, XL6, XL7: CONN_2, ~, symbol CONN_2
- removed XL13, XL18, XL28: CONN_1, ~, symbol CONN_1
- added F10, F11, F12, F13, F14, F15, F16, F17, F18, F19, F20: FUSE0R, ~, symbol FUSE0R
- added HOLE1, HOLE2, HOLE3, HOLE4: HOLE_METALLED, symbol HOLE_METALLED
- added R1, R2: 4K7, RES_0402, symbol R
- added R19, R20, R21: 51R, RES_0603, symbol R
- added R4: 150, RES_0402, symbol R
- added XL11, XL15, XL19: CONN_1, ~, symbol CONN_1
- added XL12, XL13, XL16, XL17, XL20, XL21, XL24, XL5, XL8, XL9: CONN_3, ~, symbol CONN_3
- added XL3: CONN_4, symbol CONN_4
- R10: renamed from R7; value 330k -> 390k
- R9: renamed from R6; value 330k -> 390k
- gave numbers to parts that had none: 1
- renumbered C23 to C22, C24 to C23, C25 to C24, C26 to C25, C27 to C26, C29 to C27, C30 to C28, C22 to C29, C28 to C30, Q4 to Q3, Q3 to Q4, R8 to R11, R9 to R12, R10 to R13, R11 to R14, R12 to R15, R13 to R16, R14 to R17, R15 to R18, R1 to R3, R2 to R5, R3 to R6, R4 to R7, R5 to R8, XL9 to XL10, XL19 to XL18, XL24 to XL22, XL3 to XL4, XL4 to XL6, XL8 to XL7
Connections:
- net labels added: P_SCL, P_SDA, PeriphPwr, PeriphPwr1
- wire segments 294 -> 343
- no-connect marks 21 -> 18
Other:
- note added: "For RGB"
- note added: "For WS2812B"
- note added: "Peripheral\nI2C Pull-Ups"
- note added: "Pill"
- note added: "Pill \nConnector"
- note added: "Place resistors and fuses \nif single LED is required"
- note added: "Solder fuses \nfor WS2812B"
- moved on the sheet: B1, B2, B3, C1, C10, C11, C12, C13, C14, C15, C16, C17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
