File: HandyDevices/MotorControl/MotorControl3_hw/MotorCtrl3.sch (KiCad schematic (older format))
At the start: 35 parts

Commit message: MotorControl3 Add.
Parts:
- removed C?: C, CAP_0603, symbol C
- added C? (x8): 0.1u, CAP_0603, symbol C
- added C? (x4): 10u, CAP_0603, symbol C
- added C? (x4): 220n/16v, CAP_0603, symbol C
- added C? (x4): 10n/50v, CAP_0603, symbol C
- added C? (x16): 0.1u/50v, CAP_0603, symbol C
- added C? (x8): 100u/63v, ~, symbol CP
- added C? (x12): 100p, CAP_0603, symbol C
- added D? (x8): 1N4148, ~, symbol DIODE
- added D? (x8): LED, ~, symbol LED
- added F? (x4): FUSE0R, ~, symbol FUSE0R
- added R? (x4): 32K, RES_0603, symbol R
- added R? (x4): 2K7, RES_0603, symbol R
- added R? (x12): 39K, RES_0603, symbol R
- added R? (x8): R, RES_0603, symbol R
- added U? (x4): L6470, ~, symbol L6470
- added XL? (x8): CONN_2, ~, symbol CONN_2
Connections:
- net labels added: +VS, ADC_1, ADC_2, ADC_3, ADC_4, BUSY/SYNC_1, BUSY/SYNC_2, BUSY/SYNC_3, BUSY/SYNC_4, CK_1, CK_2, CK_3, CK_4, CS_1, CS_2, CS_3, CS_4, FLAG_1, FLAG_2, FLAG_3, FLAG_4, SDI_1, SDI_2, SDI_3, SDI_4, SDO_1, SDO_2, SDO_3, SDO_4, STBY/RST_1, STBY/RST_2, STBY/RST_3, STBY/RST_4, STCK_1, STCK_2, STCK_3, STCK_4, SW_1, SW_2, SW_3, SW_4, Vdd, Vs
- wire segments 130 -> 444
- no-connect marks 1 -> 9

Commit message: Deleted ISO IC's.
Parts:
- removed DD?: STM32F405RX-64, ~, symbol STM32F405RX-64
- removed XL?: CONN_10, ~, symbol CONN_10
- added BZ?: BUZZER, ~, symbol BUZZER
- added C? (x2): C, CAP_0603, symbol C
- added C? (x2): 0.1u, CAP_0603, symbol C
- added C?: 10u, CAP_0603, symbol C
- added DD?: STM32F407VX-100, ~, symbol STM32F407VX-100
- added Q?: MMBT2222, ~, symbol NPN
- added Q?: LED_RGB, ~, symbol LED_RGB
- added R? (x2): R, RES_0603, symbol R
- added R? (x4): 51R, RES_0603, symbol R
- added XL?: CONN_2, ~, symbol CONN_2
- added XL?: CONN_NOKIA_LCD24, ~, symbol CONN_NOKIA_LCD24
- added XL?: CONN_5, ~, symbol CONN_5
- added XL?: CONN_3, ~, symbol CONN_3
- added XL?: CONN_4, ~, symbol CONN_4
- added XL?: CONN_16, ~, symbol CONN_16
- C?: value C -> 10n
- R?: value R -> 512K
Connections:
- net labels added: Buzzer, BuzzerOut, LCD_BCKLT, LCD_DA0, LCD_DA1, LCD_DA2, LCD_DA3, LCD_DA4, LCD_DA5, LCD_DA6, LCD_DA7, LCD_DC, LCD_EFF, LCD_RD, LCD_WR, LCD_XCS, LCD_XRES, LED_BLUE, LED_GREEN, LED_RED, OPT_LIMITER1, OPT_LIMITER2, OPT_LIMITER3, OPT_LIMITER4, PA0, PA10, PA15, PB12, PB3, PB5, PB8, PC13, PC14, PC15, PC5, PD11, PD3, PD7, PE15, RX3, SPI2_MISO, SPI2_MOSI, SPI2_SCK, STEP_CLK_1, STEP_CLK_2, STEP_CLK_3, STEP_CLK_4, TX3, Vacuum1, Vacuum2, Vacuum3
- net labels removed: CK_1, CK_2, CK_3, CK_4, CS_1, CS_2, CS_3, CS_4, EXT_STEP_CLOCK, EXT_VDD, SDI_1, SDO_1, SDO_2, SDO_3, SDO_4, STCK_1, STCK_2, STCK_3, STCK_4
- wire segments 444 -> 592
Other:
- note added: "Analog Power"
- note added: "Bootloader"
- note added: "Buzzer\n"
- note added: "CPU\n"
- note added: "LCD"
- note added: "LED\n"
- note added: "MOTOR DRIVER ICs\n"
- note added: "Perepherial"
- note added: "Sync output for STEP_CLK\nPA0 - SYNC_1\nPA15 - SYNC_2\nPC5 - SYNC_3\nPC13 - SYNC_4"
- note added: "TIM1 Ch4 - STEP CLK 1\n"
- note added: "TIM11 Ch1 - LCD Bcklt\n"
- note added: "TIM2 Ch2 - STEP CLK 2\n"
- note added: "TIM3 Ch1 - STEP CLK 3\n"
- note added: "TIM4 Ch3 - STEP CLK 4\n"
- note added: "TIM8 Ch1..Ch3 - RGB LED\n"
- note added: "TIM8 Ch4 - Buzzer\n"
- note added: "USB & Digital Power\n"
- note removed: "MOTOR_CONN\n"
- moved on the sheet: C?, D?, Q?, R?, SW?, U?, XL?, XTAL?

Commit message: + Added reset button.
Parts:
- added C?: 0.1u, CAP_0603, symbol C
- added R?: 100K, RES_0603, symbol R
- added SW?: BUTTON, ~, symbol BUTTON
- added XL?: CONN_3, ~, symbol CONN_3
- added XL?: CONN_2, ~, symbol CONN_2
- XL?: value CONN_2 -> MTR1_A
- XL?: value CONN_2 -> MTR1_B
- XL?: value CONN_2 -> MTR2_A
- XL?: value CONN_2 -> MTR2_B
- XL?: value CONN_2 -> MTR3_A
- XL?: value CONN_2 -> MTR3_B
- XL?: value CONN_2 -> MTR4_A
- XL?: value CONN_2 -> MTR4_B
- XL?: value CONN_2 -> +Vs
Connections:
- net labels added: DAC1, NRST, RX2, TX2
- net labels removed: MOTOR_BUSY, MOTOR_FLAG, MOTOR_STBY/RST
- wire segments 592 -> 606
- no-connect marks 9 -> 8
Other:
- note added: "Reset\n"
- moved on the sheet: BZ?, C?, D?, Q?, R?, SW?, U?, XL?, XTAL?

Commit message: * Sch ready
Parts:
- removed F? (x4): FUSE0R, ~, symbol FUSE0R
- removed XL? (x2): CONN_5, ~, symbol CONN_5
- removed XL?: CONN_4, ~, symbol CONN_4
- removed XL?: CONN_16, ~, symbol CONN_16
- added C16: 1n, CAP_0603, symbol C
- added C19: 1u, CAP_0603, symbol C
- added C5: 0.1u, CAP_0603, symbol C
- added C8: 4u7, CAP_0603, symbol C
- added C85: 10u, CAP_0603, symbol C
- added DA2: LD1117, ~, symbol LD1117
- added F1: FUSE0R, ~, symbol FUSE0R
- added HOLE1, HOLE10, HOLE11, HOLE12, HOLE13, HOLE14, HOLE2, HOLE3, HOLE4, HOLE5, HOLE6, HOLE7, HOLE8, HOLE9: HOLE_METALLED, symbol HOLE_METALLED
- added XL10, XL11, XL12, XL13: CONN_3, ~, symbol CONN_3
- added XL14, XL15, XL16, XL17, XL18, XL21, XL9: CONN_2, ~, symbol CONN_2
- added XL19: CONN_12, ~, symbol CONN_12
- added XL20: CONN_4, ~, symbol CONN_4
- C13, C18: renamed from C?; value C -> 27pF
- C2, C3: renamed from C?; value C -> 0.1u
- R10: renamed from R?; value R -> 1k
- R11, R12, R19, R20, R21, R22, R23, R24: renamed from R?; value R -> 510R
- R2: renamed from R?; value R -> 22R
- R3: renamed from R?; value R -> 510
- R34, R36, R38, R40: renamed from R?; value 32K -> 33k
- R35, R37, R39, R41: renamed from R?; value 2K7 -> 4k7
- XTAL1: renamed from XTAL?; value CRYSTAL_H -> 8MHz
- gave numbers to parts that had none: 142
Connections:
- net labels added: +12V, OUT1_1A, OUT1_1B, OUT1_2A, OUT1_2B, OUT2_1A, OUT2_1B, OUT2_2A, OUT2_2B, OUT3_1A, OUT3_1B, OUT3_2A, OUT3_2B, OUT4_1A, OUT4_1B, OUT4_2A, OUT4_2B, PC9, Vdd1, Vdd2, Vdd3, Vdd4
- net labels removed: +VS, PB8, PC13, PD11, PD3, PD7, Vdd, Vs
- wire segments 606 -> 640
Other:
- note added: "Radiator holes"
- note added: "TIM10 Ch1 - Buzzer\n"
- note removed: "Sync output for STEP_CLK\nPA0 - SYNC_1\nPA15 - SYNC_2\nPC5 - SYNC_3\nPC13 - SYNC_4"
- note removed: "TIM8 Ch4 - Buzzer\n"
- moved on the sheet: Q3, R13, R14, R15, XL22, XL23, XL24, XL25, XL26, XL27, XL28, XL29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

Commit message: + Footprint assigned to components. Check values and e.t.c.
Parts:
- removed XL19: CONN_12, ~, symbol CONN_12
- added XL19: CONN_10, ~, symbol CONN_10
- added XL30, XL31: CONN_3, ~, symbol CONN_3
- C20, C34, C53, C55, C57, C85: footprint CAP_0603 -> CAP_0805
- C35, C54, C56, C58: value 100u/63v -> 4u7/63v
- C37, C64, C66, C68: footprint CAP_0603 -> CAP_1206
Connections:
- wire segments 640 -> 648
Other:
- moved on the sheet: C16, C19, C5, C8, DA2, HOLE1, HOLE10, HOLE11, HOLE12, HOLE13, HOLE14, HOLE2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

Commit message: * USB connector replaced with B type
Parts:
- removed XL1: USB_MINI_B, ~, symbol USB_MINI_B
- added XL1: USB_B, ~, symbol USB_B
Connections:
- wire segments 648 -> 647
Other:
- moved on the sheet: C1, R1
Changed lines of the file:
@@
 Sheet 1 1
 Title "Motor Control v.3"
-Date "14 apr 2014"
+Date "16 apr 2014"
 Rev ""
 Comp ""
@@
 $EndComp
 $Comp
-L USB_MINI_B XL1
-U 1 1 5301D1D5
-P 1250 14150
-F 0 "XL1" H 1050 14600 60  0000 C CNN
-F 1 "USB_MINI_B" H 1150 14500 60  0000 C CNN
-F 2 "~" H 1250 14150 60  0000 C CNN
-F 3 "~" H 1250 14150 60  0000 C CNN
-	1    1250 14150
-	1    0    0    -1
-$EndComp
-$Comp
 L R R1
 U 1 1 5301D1E4
-P 1100 15000
-F 0 "R1" V 1180 14850 50  0000 C CNN
-F 1 "512K" V 1100 15000 50  0000 C CNN
-F 2 "RES_0603" V 1180 15100 28  0000 C CNN
-F 3 "~" H 1100 15000 60  0000 C CNN
-	1    1100 15000
+P 1100 14900
+F 0 "R1" V 1180 14750 50  0000 C CNN
+F 1 "512K" V 1100 14900 50  0000 C CNN
+F 2 "RES_0603" V 1180 15000 28  0000 C CNN
+F 3 "~" H 1100 14900 60  0000 C CNN
+	1    1100 14900
 	1    0    0    -1
 $EndComp
@@
 L C C1
 U 1 1 5301D1F3
-P 1350 15000
-F 0 "C1" H 1250 14900 50  0000 L CNN
-F 1 "10n" H 1250 15100 50  0000 L CNN
-F 2 "CAP_0603" V 1450 14850 28  0000 C BNN
-F 3 "~" H 1350 15000 60  0000 C CNN
-	1    1350 15000
+P 1350 14900
+F 0 "C1" H 1250 14800 50  0000 L CNN
+F 1 "10n" H 1250 15000 50  0000 L CNN
+F 2 "CAP_0603" V 1450 14750 28  0000 C BNN
+F 3 "~" H 1350 14900 60  0000 C CNN
+	1    1350 14900
 	1    0    0    -1
 $EndComp
@@
 L GND #PWR08
 U 1 1 5301D314
-P 1100 15400
-F 0 "#PWR08" H 1190 15380 30  0001 C CNN
-F 1 "GND" H 1100 15320 30  0001 C CNN
-F 2 "" H 1100 15400 60  0000 C CNN
-F 3 "" H 1100 15400 60  0000 C CNN
-	1    1100 15400
+P 1100 15300
+F 0 "#PWR08" H 1190 15280 30  0001 C CNN
+F 1 "GND" H 1100 15220 30  0001 C CNN
+F 2 "" H 1100 15300 60  0000 C CNN
+F 3 "" H 1100 15300 60  0000 C CNN
+	1    1100 15300
 	1    0    0    -1
 $EndComp
@@
 	7750 13400 7750 13450
 Wire Wire Line
-	1100 14650 1100 14750
+	1100 14550 1100 14650
 Wire Wire Line
-	1100 14700 1350 14700
+	1100 14600 1350 14600
 Wire Wire Line
-	1350 14700 1350 14800
-Connection ~ 1100 14700
+	1350 14600 1350 14700
+Connection ~ 1100 14600
 Wire Wire Line
-	1100 15250 1100 15400
+	1100 15150 1100 15300
 Wire Wire Line
-	1100 15300 1350 15300
+	1100 15200 1350 15200
 Wire Wire Line
-	1350 15300 1350 15200
-Connection ~ 1100 15300
+	1350 15200 1350 15100
+Connection ~ 1100 15200
 Wire Wire Line
 	1450 13950 2000 13950
@@
 	1600 14250 1600 14500
 Wire Wire Line
-	1600 14350 1450 14350
-Connection ~ 1600 14350
-Wire Wire Line
 	2500 14800 2500 14950
 Wire Wire Line
@@
 	1    0    0    -1
 $EndComp
+$Comp
+L USB_B XL1
+U 1 1 534E37B2
+P 1250 14150
+F 0 "XL1" H 1050 14600 60  0000 C CNN
+F 1 "USB_B" H 1150 14500 60  0000 C CNN
+F 2 "~" H 1250 14150 60  0000 C CNN
+F 3 "~" H 1250 14150 60  0000 C CNN
+	1    1250 14150
+	1    0    0    -1
+$EndComp

Commit message: + PCB
Parts:
- removed XL19: CONN_10, ~, symbol CONN_10
- added XL32: CONN_4, ~, symbol CONN_4
Connections:
- net labels removed: PA10, PA15, PB12, PB3, PB5, PC14, PC15, PC5, PE15
- wire segments 647 -> 633
- no-connect marks 8 -> 17
Other:
- moved on the sheet: Q3

Commit message: 
Parts:
- removed Q3: LED_RGB, ~, symbol LED_RGB
- removed R13, R14, R15: 51R, RES_0603, symbol R
- removed SW2: BUTTON, ~, symbol BUTTON
- removed XL10, XL11, XL12, XL13, XL30, XL31, XL6, XL7: CONN_3, ~, symbol CONN_3
- removed XL14, XL15, XL16, XL17, XL18, XL21, XL8, XL9: CONN_2, ~, symbol CONN_2
- removed XL20, XL32: CONN_4, ~, symbol CONN_4
- removed XL22: MTR4_A, ~, symbol CONN_2
- removed XL23: MTR4_B, ~, symbol CONN_2
- removed XL24: MTR3_A, ~, symbol CONN_2
- removed XL25: MTR3_B, ~, symbol CONN_2
- removed XL26: MTR1_A, ~, symbol CONN_2
- removed XL27: MTR1_B, ~, symbol CONN_2
- removed XL28: MTR2_A, ~, symbol CONN_2
- removed XL29: MTR2_B, ~, symbol CONN_2
- added C?: 0.1u, symbol C
- added C?: 0.1u, CAP_0603, symbol C
- added DD?: M24C04, SO8E, symbol EEPROM_I2C
- added R? (x2): 4k7, symbol R
- added TP? (x24): TESTPOINT, symbol TESTPOINT
- added XL?: CONN_MICROSD, symbol CONN_MICROSD
- added XL? (x4): CONN_4, ~, symbol CONN_4
- added XL? (x4): CONN_4X2, ~, symbol CONN_4X2
- added XL?: CONN_2, ~, symbol CONN_2
- R8: value 100K -> 10k
Connections:
- net labels added: GPIO1, GPIO2, GPIO3, I2C_SCL, I2C_SDA, LIMITER5, LIMITER6, LIMITER7, LIMITER8, SD_CLK, SD_CMD, SD_DAT0, SD_DAT1, SD_DAT2, SD_DAT3, STBY/RST
- net labels removed: DAC1, LED_BLUE, LED_GREEN, LED_RED, NRST, OPT_LIMITER1, OPT_LIMITER2, OPT_LIMITER3, OPT_LIMITER4, PA0, PC9, RX2, RX3, STBY/RST_1, STBY/RST_2, STBY/RST_3, STBY/RST_4, TX2, TX3, Vacuum3
- wire segments 633 -> 666
- no-connect marks 17 -> 23
Other:
- note added: "Buzzer"
- note added: "I2C Addr = 1010 (A2)(A1)(A0) in case of 1 or 2 kBit,\nI2C Addr = 1010 (A2)(A1) in case of 4 kBit.\nA2, A1, A0 are read as 0 when left floating"
- note added: "I2C pull-ups"
- note added: "Limiters"
- note added: "SD card"
- note removed: "Buzzer\n"
- note removed: "LED\n"
- note removed: "LIMITERS\n"
- note removed: "Perepherial"
- note removed: "TIM8 Ch1..Ch3 - RGB LED\n"
- moved on the sheet: BZ1, C1, C12, C15, C16, C19, C27, C28, C29, C30, C31, C32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
