File: Lockets/SeidheLocket/SeidheLocket_hw/SeidheLocket.kicad_pcb (KiCad board)
At the start: 2 copper layers, 101 x 24 mm, 49 parts, among them M1 MOTOR_PAD, Q1 MMBT2222, Q2 LED_RGB 5050, SW1 BUTTON

Commit message: * SeidheLocket final PCB + GERBER
Parts:
- ANT1: footprint ANT_MEANDER868_16MM -> ANT_868_SEIDHE
- moved RP2 21.2 mm to (236.2, 170.0)
- moved RP1 21.0 mm to (174.9, 191.9)
- moved C6 1.08 mm to (229.0, 183.0)
- moved C1 1.00 mm to (186.4, 187.1), turned to 90 degrees
- moved XTAL1 0.89 mm to (231.4, 186.0)
- moved C10 0.72 mm to (234.4, 185.8)
- moved C9 0.72 mm to (228.4, 185.8)
- moved TP1 0.72 mm to (225.0, 182.8)
- moved DD2 0.72 mm to (228.8, 178.8)
- moved BLN1 0.72 mm to (233.0, 179.1)
- moved C11 0.72 mm to (224.0, 180.6)
- moved C3 0.72 mm to (231.2, 174.2)
- moved C5 0.72 mm to (232.0, 182.6)
- moved C7 0.72 mm to (224.0, 179.0)
- moved C8 0.72 mm to (228.0, 174.2)
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Routing:
- net GND: track 0.00 -> 488.3 mm, vias 0 -> 87
- net +3.3V: track 0.00 -> 137.1 mm, vias 0 -> 10
- net N-0000012: track 0.00 -> 37.0 mm, vias 0 -> 2
- net +BATT: track 0.00 -> 32.3 mm
- net N-0000020: track 0.00 -> 30.9 mm, vias 0 -> 2
- net /CC_GDO2: track 0.00 -> 25.0 mm, vias 0 -> 2
- net /CC_MOSI: track 0.00 -> 21.2 mm
- net /CC_MISO: track 0.00 -> 20.5 mm
- net /CC_CS: track 0.00 -> 19.8 mm
- net /CC_SCK: track 0.00 -> 19.2 mm, vias 0 -> 2
- net /CC_GDO0: track 0.00 -> 18.5 mm, vias 0 -> 2
- net /GREEN_LED: track 0.00 -> 16.5 mm
- net N-000008: track 0.00 -> 15.0 mm, vias 0 -> 1
- net N-0000037: track 0.00 -> 14.5 mm, vias 0 -> 2
- net /BLUE_LED: track 0.00 -> 13.9 mm, vias 0 -> 2
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- added copper zone on B.Cu, net GND
- added copper zone on F.Cu, net GND
Other:
- board size 101 x 24 mm -> 99.9 x 24 mm
