File: HandyDevices/BmstuCtrl/BmstuCtrl_hw/BmstuCtrl.sch (KiCad schematic (older format))
At the start: 38 parts

Commit message: * Sch seems completed
Parts:
- removed C? (x2): 20pF, CAP_0603, symbol C
- removed R?: 220R, RES_0603, symbol R
- removed XTAL?: 12.0MHz, 0532, symbol CRYSTAL_H
- added C10, C11, C12, C9: 0.1u, CAP_0603, symbol C
- added D1: LED, ~, symbol LED
- added DA3, DA4, DA5, DA6: MC74VHC1, symbol MC74VHC1
- added R1: 100R, RES_0603, symbol R
- added R3: 10k, RES_0603, symbol R
- gave numbers to parts that had none: 34
Connections:
- net labels added: OutputEn, PATH2_1_IN, PATH2_2_IN, PATH3_1_IN, PATH3_2_IN
- wire segments 133 -> 155
- no-connect marks 16 -> 34
Other:
- note added: "Holes & ref points"
- note added: "Output buffers\nDisabled by default"
- note added: "Power & Signal Connectors"
- note added: "Power input"
- note added: "RS-485 interface"
- moved on the sheet: C4, C8, DA1, HOLE1, HOLE2, HOLE3, HOLE4, RP1, RP2, XL1, XL10, XL2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

Commit message: Bmstu Ctrl hw completed
Parts:
- removed RP1, RP2: REFPOINT, symbol REFPOINT
- removed XL10, XL9: CONN_8, ~, symbol CONN_8
- removed XL6, XL8: CONN_4, ~, symbol CONN_4
- removed XL7: CONN_2, ~, symbol CONN_2
- added D2, D3, D4, D5: LED, ~, symbol LED
- added HOLE10, HOLE11, HOLE12, HOLE13, HOLE14, HOLE5, HOLE6, HOLE7, HOLE9: HOLE_METALLED, symbol HOLE_METALLED
- added R2, R3, R4, R5: 1k, RES_0603, symbol R
- added R8: 150R, RES_0603, symbol R
- added XL10, XL11, XL12, XL13, XL14, XL15, XL16, XL17, XL18, XL19, XL20, XL21, XL22, XL23, XL24, XL25, XL26, XL27, XL28, XL29, XL30, XL31, XL5, XL6, XL7, XL8: CONN_GOST_1, ~, symbol CONN_GOST_1
- renumbered D2 to D6, D3 to D7, R2 to R6, R3 to R7, XL5 to XL9
Connections:
- wire segments 155 -> 179
Other:
- note added: "Holes"
- note removed: "Holes & ref points"
- moved on the sheet: C10, C11, C12, C9, DA3, DA4, DA5, DA6, HOLE1, HOLE2, HOLE3, HOLE4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
